File: attiny48.kicad_pcb (KiCad board)
At the start: 2 copper layers, 20.3 x 19.3 mm, 11 parts, among them J1 POWER, J2 PORTA, J3 PORTB, J4 PORTC, J5 PORTD, U1 ATtiny88-AU

Commit message: Adds symbols to PCB
Parts:
- J2: footprint Connector_PinHeader_1.00mm:PinHeader_1x04_P1.00mm_Vertical -> Connector_PinSocket_1.00mm:PinSocket_1x04_P1.00mm_Vertical
- J3, J4, J5: footprint Connector_PinHeader_1.00mm:PinHeader_1x08_P1.00mm_Vertical -> Connector_PinSocket_1.00mm:PinSocket_1x08_P1.00mm_Vertical
